File: flight_controller.kicad_pcb (KiCad board)
At the start: 4 copper layers, 59 x 59 mm, 65 parts, among them J1 Conn_01x03_Pin, J2 Conn_01x02_Socket, J3 USB_C_Receptacle_USB2.0_16P, J4 Conn_01x03_Pin, J5 Conn_01x03_Pin, J6 Conn_01x03_Pin, J7 Conn_01x03_Pin, J8 Conn_01x05_Socket, J9 Conn_01x04_Socket, Q1 AO3401A, U1 STM32F405RGTx, U2 AP63205WU, U3 TLV70233_SOT23-5, U4 USBLC6-2SC6, U5 LPS22HB, Y1 8MHz Crystal_GND24

Commit message: first commit
Parts:
- 3V3, 5V, GND: footprint TestPoint:TestPoint_Pad_D1.0mm -> flight_controller:TestPoint_Pad_D1.0mm
- AC1: footprint Package_LGA:LGA-14_3x2.5mm_P0.5mm_LayoutBorder3x4y -> flight_controller:LGA-14_3x2.5mm_P0.5mm_LayoutBorder3x4y
- C1, C11, C12, C13, C15, C2, C21, C22, C23, C24, C25, C3, C4, C5, C7: footprint Capacitor_SMD:C_0402_1005Metric -> flight_controller:C_0402_1005Metric
- C10, C14, C20, C6, C9: footprint Capacitor_SMD:C_0805_2012Metric -> flight_controller:C_0805_2012Metric
- C16, C17: footprint Capacitor_SMD:C_1206_3216Metric -> flight_controller:C_1206_3216Metric
- C18, C19, C8: footprint Capacitor_SMD:C_0603_1608Metric -> flight_controller:C_0603_1608Metric
- D1: footprint Diode_SMD:D_SMC -> flight_controller:D_SMC
- D2, D3: footprint LED_SMD:LED_0805_2012Metric -> flight_controller:LED_0805_2012Metric
- FB1: footprint Inductor_SMD:L_0805_2012Metric -> flight_controller:L_0805_2012Metric
- H1, H2, H3, H4: footprint MountingHole:MountingHole_3.7mm_Pad_Via -> flight_controller:MountingHole_3.7mm_Pad_Via
- J1, J4, J5, J6, J7: footprint Connector_PinHeader_2.54mm:PinHeader_1x03_P2.54mm_Vertical -> flight_controller:PinHeader_1x03_P2.54mm_Vertical
- J2: footprint Connector_PinSocket_2.54mm:PinSocket_1x02_P2.54mm_Vertical -> flight_controller:PinSocket_1x02_P2.54mm_Vertical
- J3: footprint Connector_USB:USB_C_Receptacle_HRO_TYPE-C-31-M-12 -> flight_controller:USB_C_Receptacle_HRO_TYPE-C-31-M-12
- J8: footprint Connector_PinSocket_2.54mm:PinSocket_1x05_P2.54mm_Vertical -> flight_controller:PinSocket_1x05_P2.54mm_Vertical
- J9: footprint Connector_PinSocket_2.54mm:PinSocket_1x04_P2.54mm_Vertical -> flight_controller:PinSocket_1x04_P2.54mm_Vertical
- L1: footprint Inductor_SMD:L_Sunlord_MWSA0503S -> flight_controller:L_Sunlord_MWSA0503S
- Q1: footprint Package_TO_SOT_SMD:SOT-23 -> flight_controller:SOT-23
- R1, R10, R11, R2, R3, R4, R5, R6, R7, R8, R9: footprint Resistor_SMD:R_0402_1005Metric -> flight_controller:R_0402_1005Metric
- U1: footprint Package_QFP:LQFP-64_10x10mm_P0.5mm -> flight_controller:LQFP-64_10x10mm_P0.5mm
- U2: footprint Package_TO_SOT_SMD:TSOT-23-6 -> flight_controller:TSOT-23-6
- U3: footprint Package_TO_SOT_SMD:SOT-23-5 -> flight_controller:SOT-23-5
- U4: footprint Package_TO_SOT_SMD:SOT-23-6 -> flight_controller:SOT-23-6
- U5: footprint Package_LGA:ST_HLGA-10_2x2mm_P0.5mm_LayoutBorder3x2y -> flight_controller:ST_HLGA-10_2x2mm_P0.5mm_LayoutBorder3x2y
- Y1: footprint Crystal:Crystal_SMD_3225-4Pin_3.2x2.5mm -> flight_controller:Crystal_SMD_3225-4Pin_3.2x2.5mm
